Commit message: add jetson mouse urdf

File: ros2_docker/colcon_ws/src/jetsonmouse_description/urdf/body/body.urdf.xacro (robot description, xacro)
@@ -1,5 +1,4 @@
 <?xml version="1.0"?>
 <robot xmlns:xacro="http://ros.org/wiki/xacro">
-  <xacro:include filename="$(find raspimouse_description)/urdf/body/body.gazebo.xacro" />
   <xacro:macro name="base" params="parent *joint_origin">
     <joint name="base_joint" type="fixed">
@@ -11,11 +10,8 @@
       <visual>
         <geometry>
-          <mesh filename="package://raspimouse_description/meshes/dae/body/raspimouse_body.dae" />
+          <mesh filename="package://jetsonmouse_description/meshes/dae/jetsonmouse_body.dae" />
         </geometry>
       </visual>
       <collision>
-        <!-- <geometry> -->
-          <!-- <mesh filename="package://raspimouse_description/meshes/dae/body/raspimouse_body.dae" /> -->
-        <!-- </geometry> -->
         <origin rpy="0 0 0" xyz="0.005 0 0.040" />
         <geometry>
@@ -24,11 +20,34 @@
       </collision>
       <inertial>
+        <origin xyz="-0.005075 -0.000427 0.029879" />
         <mass value="0.7186" />
-        <origin xyz="-0.005075 0.0 0.03" />
-        <xacro:box_inertia m="0.7" x="0.1" y="0.08" z="0.08" />
-        <!-- <origin xyz="-0.005075 -0.000427 0.029879" /> -->
-        <!-- <inertia ixx="0.001238161833" ixy="0.000000904986" iyy="0.001368529369"
-                  ixz="0.000100297310" iyz="0.000022118177" izz="0.000784319117" /> -->
+        <inertia ixx="0.001238161833" ixy="0.000000904986" iyy="0.001368529369" ixz="0.000100297310" iyz="0.000022118177" izz="0.000784319117" />
       </inertial>
+    </link>
+    <joint name="right_camera_joint" type="fixed">
+      <origin xyz="0.063912 -0.0275 0.080798" rpy="${radians(110)} 0 ${radians(90)}" />
+      <parent link="base_link" />
+      <child link="right_camera_link" />
+    </joint>
+    <link name="right_camera_link">
+      <collision>
+          <origin xyz="0 0 0.012" />
+          <geometry>
+            <cylinder radius="0.008" length="0.015" />
+          </geometry>
+      </collision>
+    </link>
+    <joint name="left_camera_joint" type="fixed">
+      <origin xyz="0.063912 0.0275 0.080798" rpy="${radians(110)} 0 ${radians(90)}" />
+      <parent link="base_link" />
+      <child link="left_camera_link" />
+    </joint>
+    <link name="left_camera_link">
+      <collision>
+          <origin xyz="0 0 0.012" />
+          <geometry>
+            <cylinder radius="0.008" length="0.015" />
+          </geometry>
+      </collision>
     </link>
   </xacro:macro>

File: ros2_docker/colcon_ws/src/jetsonmouse_description/urdf/camera/camera.gazebo.xacro (robot description, xacro)
@@ -2,10 +2,7 @@
 <robot name="csi_camera" xmlns:xacro="http://ros.org/wiki/xacro">
   <xacro:macro name="camera_gazebo" params="camera_name camera_link robot_namespace robotdescription_namespace">
-    <gazebo reference="${camera_link}">
-      <material>Gazebo/FlatBlack</material>
-    </gazebo>
     <link name="${camera_link}_tf_origin" />
     <joint name="${camera_link}_tf_joint" type="fixed">
-      <origin xyz="0 0 0" rpy="0 0 0" />
+      <origin xyz="0 0 0" rpy="0 -1.57 -1.57" />
       <parent link="${camera_link}" />
       <child link="${camera_link}_tf_origin" />
@@ -13,9 +10,9 @@
     <gazebo reference="${camera_link}_tf_origin">
       <sensor type="camera" name="${camera_name}">
-        <visualize>$(arg camera_visual)</visualize>
+        <visualize>true</visualize>
         <update_rate>30.0</update_rate>
         <camera name="${camera_name}">
           <pose>0 0 0 0 0 0</pose>
-          <horizontal_fov>1.39626</horizontal_fov> <!-- 80deg -->
+          <horizontal_fov>2.79253</horizontal_fov> <!-- 160deg -->
           <image>
             <width>800</width>
@@ -25,5 +22,5 @@
           <clip>
             <near>0.03</near>
-            <far>3</far>
+            <far>1</far>
           </clip>
           <noise>

File: ros2_docker/colcon_ws/src/jetsonmouse_description/urdf/common.xacro (robot description, xacro)
@@ -4,8 +4,8 @@
   <xacro:property name="wheel_length" value="0.010" />
   <xacro:property name="wheel_mass" value="0.0113" />
-  <xacro:property name="wheel_separation" value="0.0935" />
+  <xacro:property name="wheel_separation" value="0.0925" />
   <!-- PROPERTY LIST -->
   <!-- All units in m-kg-s-radians unit system -->
-  <xacro:property name="M_PI" value="3.1415926535897932" />
+  <xacro:property name="M_PI" value="3.1415926535897931" />
   <!-- Inertial macros. Units are kg*m^2 -->
   <xacro:macro name="box_inertia" params="m x y z">
@@ -20,7 +20,7 @@
   </xacro:macro>
   <xacro:macro name="sphere_inertia" params="m r">
-    <inertia ixx="${m*r*r*2/5}" ixy="0" ixz="0"
-             iyy="${m*r*r*2/5}" iyz="0"
-             izz="${m*r*r*2/5}" />
+    <inertia ixx="${m*r*r/5}" ixy="0" ixz="0"
+             iyy="${m*r*r/5}" iyz="0"
+             izz="${m*r*r/5}" />
   </xacro:macro>
 </robot>

File: ros2_docker/colcon_ws/src/jetsonmouse_description/urdf/sensors/lightsens.gazebo.xacro (robot description, xacro)
@@ -1,7 +1,6 @@
 <?xml version="1.0"?>
 <robot xmlns:xacro="http://ros.org/wiki/xacro">
-  <xacro:macro name="lightsensor_gazebo" params="prefix base_rad rad_range min_range max_range robotdescription_namespace robot_namespace">
-    <gazebo reference="${prefix}_lightsensor_link">
-      <material>Gazebo/Gray</material>
+  <xacro:macro name="lightsensor_gazebo" params="prefix base_rad rad_range min_range max_range robot_namespace">
+    <gazebo reference="${prefix}">
       <sensor type="ray" name="${prefix}_lightsensor">
         <pose>0 0 0 0 0 0</pose>
@@ -31,5 +30,5 @@
           <robotNamespace>${robot_namespace}</robotNamespace>
           <topicName>${prefix}_scan</topicName>
-          <frameName>${robotdescription_namespace}${prefix}</frameName>
+          <frameName>${prefix}</frameName>
         </plugin>
       </sensor>

File: ros2_docker/colcon_ws/src/jetsonmouse_description/urdf/sensors/lightsens.urdf.xacro (robot description, xacro)
@@ -1,21 +1,19 @@
 <?xml version="1.0"?>
 <robot name="light_sensor" xmlns:xacro="http://ros.org/wiki/xacro">
-  <xacro:include filename="$(find raspimouse_description)/urdf/common.xacro" />
-  <xacro:include filename="$(find raspimouse_description)/urdf/sensors/lightsens.gazebo.xacro" />
+  <xacro:include filename="$(find jetsonmouse_description)/urdf/common.xacro" />
+  <xacro:include filename="$(find jetsonmouse_description)/urdf/sensors/lightsens.gazebo.xacro" />
   <xacro:macro name="light_sensor" params="prefix parent *joint_origin">
     <joint name="${prefix}_joint" type="fixed">
       <xacro:insert_block name="joint_origin" />
       <parent link="${parent}" />
-      <child link="${prefix}_lightsensor_link" />
+      <child link="${prefix}" />
     </joint>
-    <link name="${prefix}_lightsensor_link">
+    <link name="${prefix}">
       <visual>
         <geometry>
           <box size="0.01 0.005 0.007" />
         </geometry>
-        <material name="Gray">
-          <color rgba="0.2 0.2 0.2 1" />
-        </material>
       </visual>
+      <material name="Gray" />
       <inertial>
         <mass value="0.000001" />

File: ros2_docker/colcon_ws/src/jetsonmouse_description/urdf/wheel/diffdrive.gazebo.xacro (robot description, xacro)
@@ -1,5 +1,5 @@
 <?xml version="1.0"?>
 <robot name="diffdrive_gazebo" xmlns:xacro="http://ros.org/wiki/xacro">
-  <xacro:include filename="$(find raspimouse_description)/urdf/common.xacro" />
+  <xacro:include filename="$(find jetsonmouse_description)/urdf/common.xacro" />
   <xacro:macro name="diffdrive_gazebo" params="publish_tf publish_jointstate robot_namespace">
     <gazebo>
@@ -33,11 +33,11 @@
         <wheelAcceleration>0</wheelAcceleration>
         <!-- Set to true to publish /odom (nav_msgs::Odometry), defaults to true -->
-        <publishTf>${publish_tf}</publishTf>
+        <publishTf>$(arg tf)</publishTf>
         <!-- Set to true to publish transforms for the wheel links, defaults to false -->
-        <publishWheelTF>${publish_tf}</publishWheelTF>
+        <publishWheelTF>$(arg tf)</publishWheelTF>
         <!-- Set to true to publish transforms for the odometry, defaults to true -->
-        <publishOdomTF>${publish_tf}</publishOdomTF>
+        <publishOdomTF>$(arg tf)</publishOdomTF>
         <!-- Set to true to publish sensor_msgs/JointState on /joint_states for the wheel joints, defaults to false -->
-        <publishWheelJointState>${publish_jointstate}</publishWheelJointState>
+        <publishWheelJointState>$(arg jointstate)</publishWheelJointState>
       </plugin>
     </gazebo>

File: ros2_docker/colcon_ws/src/jetsonmouse_description/urdf/wheel/wheel.urdf.xacro (robot description, xacro)
@@ -1,40 +1,27 @@
 <?xml version="1.0"?>
 <robot xmlns:xacro="http://ros.org/wiki/xacro">
-  <xacro:include filename="$(find raspimouse_description)/urdf/common.xacro" />
+  <xacro:include filename="$(find jetsonmouse_description)/urdf/common.xacro" />
   <xacro:macro name="wheel" params="prefix parent *joint_origin *joint_axis">
-    <joint name="${prefix}_wheel_joint" type="continuous">
-      <xacro:insert_block name="joint_origin" />
-      <xacro:insert_block name="joint_axis" />
-      <parent link="${parent}" />
-      <child link="${prefix}_wheel" />
-      <limit effort="70" velocity="15" />
-      <safety_controller k_velocity="10" />
-      <dynamics damping="1.0" friction="1.0" />
-    </joint>
-    <link name="${prefix}_wheel">
-      <visual>
-        <geometry>
-          <mesh filename="package://raspimouse_description/meshes/dae/wheel/raspimouse_wheel.dae" />
-        </geometry>
-      </visual>
-      <collision>
-        <!-- <geometry> -->
-        <!-- <mesh filename="package://raspimouse_description/meshes/dae/wheel/raspimouse_wheel.dae"/> -->
-        <!-- </geometry> -->
-        <origin xyz="0 0 0.003" />
+  <joint name="${prefix}_wheel_joint" type="continuous">
+    <xacro:insert_block name="joint_origin" />
+    <xacro:insert_block name="joint_axis" />
+    <parent link="${parent}" />
+    <child link="${prefix}_wheel" />
+    <limit effort="70" velocity="15" />
+    <safety_controller  k_velocity="10" />
+    <dynamics damping="1.0" friction="1.0" />
+  </joint>
+  <link name="${prefix}_wheel">
+    <visual>
+      <geometry>
+        <mesh filename="package://jetsonmouse_description/meshes/dae/jetsonmouse_wheel.dae" />
+      </geometry>
+    </visual>
+    <collision>
+      <origin xyz="0 0 0.003" />
         <geometry>
           <cylinder radius="${wheel_radius}" length="${wheel_length}" />
         </geometry>
-        <surface>
-          <friction>
-            <ode>
-              <mu>2</mu>
-              <mu2>2</mu2>
-              <slip1>0</slip1>
-              <slip2>0</slip2>
-            </ode>
-          </friction>
-        </surface>
-      </collision>
+    </collision>
       <inertial>
         <origin xyz="-0.000107 0 0.002875" />
@@ -42,5 +29,5 @@
         <inertia ixx="0.000002208187" ixy="0.000000000001" iyy="0.00000218412" ixz="0.000000004787" iyz="0.000000000003" izz="0.000004078299" />
       </inertial>
-    </link>
+  </link>
   </xacro:macro>
 </robot>
